File: Electrical/Circuit Boards/Raspberry Pi HATs/ADC HAT/HAT.kicad_pcb (KiCad board)
At the start: 2 copper layers, 65 x 56 mm, 31 parts, among them J1 CONN_01X02, J10 CONN_01X03, J11 CONN_01X03, J12 CONN_01X03, J13 CONN_01X03, J14 CONN_01X03, J15 CONN_01X03, J16 CONN_01X03, J17 CONN_01X03, J18 CONN_01X03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

Commit message: Correct missing ground on C1,C2
Connections:
- C1 pad 2: Net-(C1-Pad2) -> GND
- C2 pad 2: Net-(C1-Pad2) -> GND
Routing:
- net GND: track 13.3 -> 23.3 mm
- net Net-(C1-Pad2): track 3.43 -> 0.00 mm
Changed lines of the file:
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@@
 (kicad_pcb (version 4) (host pcbnew 4.0.6)
   (general
-    (links 83)
+    (links 84)
     (no_connects 1)
     (area 99.924999 74.924999 165.075001 131.075001)
     (thickness 1.6)
     (drawings 61)
-    (tracks 218)
+    (tracks 224)
     (zones 0)
     (modules 31)
-    (nets 29)
+    (nets 28)
   )
   (page A4)
@@
   )
   (setup
-    (last_trace_width 0.762)
+    (last_trace_width 0.25)
     (user_trace_width 0.254)
     (user_trace_width 0.381)
@@
   (net 23 "Net-(R2-Pad2)")
   (net 24 "Net-(C1-Pad1)")
-  (net 25 "Net-(C1-Pad2)")
-  (net 26 "Net-(C3-Pad1)")
-  (net 27 "Net-(J21-Pad2)")
-  (net 28 "Net-(J20-Pad3)")
+  (net 25 "Net-(C3-Pad1)")
+  (net 26 "Net-(J21-Pad2)")
+  (net 27 "Net-(J20-Pad3)")
   (net_class Default "This is the default net class."
     (clearance 0.2)
@@
     (add_net GND)
     (add_net "Net-(C1-Pad1)")
-    (add_net "Net-(C1-Pad2)")
     (add_net "Net-(C3-Pad1)")
     (add_net "Net-(J10-Pad2)")
@@
       (net 5 GND))
     (pad 20 smd rect (at 2.95 -2.925) (size 1.45 0.45) (layers F.Cu F.Paste F.Mask)
-      (net 27 "Net-(J21-Pad2)"))
+      (net 26 "Net-(J21-Pad2)"))
     (model ${KISYS3DMOD}/Housings_SSOP.3dshapes/TSSOP-20_4.4x6.5mm_Pitch0.65mm.wrl
       (at (xyz 0 0 0))
@@
       (net 24 "Net-(C1-Pad1)"))
     (pad 2 smd rect (at 1.5 0 270) (size 1 2.5) (layers F.Cu F.Paste F.Mask)
-      (net 25 "Net-(C1-Pad2)"))
+      (net 5 GND))
     (model Capacitors_SMD.3dshapes/C_1210.wrl
       (at (xyz 0 0 0))
@@
       (net 24 "Net-(C1-Pad1)"))
     (pad 2 smd rect (at 1.5 0 270) (size 1 2.5) (layers F.Cu F.Paste F.Mask)
-      (net 25 "Net-(C1-Pad2)"))
+      (net 5 GND))
     (model Capacitors_SMD.3dshapes/C_1210.wrl
       (at (xyz 0 0 0))
@@
     (fp_line (start 2.25 1.5) (end -2.25 1.5) (layer F.CrtYd) (width 0.05))
     (pad 1 smd rect (at -1.5 0 270) (size 1 2.5) (layers F.Cu F.Paste F.Mask)
-      (net 26 "Net-(C3-Pad1)"))
+      (net 25 "Net-(C3-Pad1)"))
     (pad 2 smd rect (at 1.5 0 270) (size 1 2.5) (layers F.Cu F.Paste F.Mask)
       (net 5 GND))
@@
       (net 24 "Net-(C1-Pad1)"))
     (pad 3 thru_hole oval (at 0 5.08) (size 1.7 1.7) (drill 1) (layers *.Cu *.Mask)
-      (net 28 "Net-(J20-Pad3)"))
+      (net 27 "Net-(J20-Pad3)"))
     (pad 4 thru_hole oval (at 0 7.62) (size 1.7 1.7) (drill 1) (layers *.Cu *.Mask)
-      (net 28 "Net-(J20-Pad3)"))
+      (net 27 "Net-(J20-Pad3)"))
     (model ${KISYS3DMOD}/Pin_Headers.3dshapes/Pin_Header_Straight_1x04_Pitch2.54mm.wrl
       (at (xyz 0 0 0))
@@
       (net 5 GND))
     (pad 2 thru_hole oval (at 0 2.54) (size 1.7 1.7) (drill 1) (layers *.Cu *.Mask)
-      (net 27 "Net-(J21-Pad2)"))
+      (net 26 "Net-(J21-Pad2)"))
     (pad 3 thru_hole oval (at 0 5.08) (size 1.7 1.7) (drill 1) (layers *.Cu *.Mask)
-      (net 26 "Net-(C3-Pad1)"))
+      (net 25 "Net-(C3-Pad1)"))
     (model ${KISYS3DMOD}/Pin_Headers.3dshapes/Pin_Header_Straight_1x03_Pitch2.54mm.wrl
       (at (xyz 0 0 0))
@@
   (segment (start 125.603 104.013) (end 128.143 104.013) (width 0.762) (layer B.Cu) (net 3))
   (segment (start 128.143 104.013) (end 130.683 104.013) (width 0.762) (layer B.Cu) (net 3))
-  (segment (start 112.903 109.093) (end 111.125 109.093) (width 0.762) (layer B.Cu) (net 4) (status 400000))
+  (segment (start 112.903 109.093) (end 111.125 109.093) (width 0.762) (layer B.Cu) (net 4))
   (via (at 109.728 107.696) (size 1.016) (drill 0.67818) (layers F.Cu B.Cu) (net 4))
   (segment (start 111.125 109.093) (end 109.728 107.696) (width 0.762) (layer B.Cu) (net 4))
-  (segment (start 133.448 96.651) (end 133.448 98.2) (width 0.254) (layer F.Cu) (net 4) (status 400000))
+  (segment (start 133.448 96.651) (end 133.448 98.2) (width 0.254) (layer F.Cu) (net 4))
   (segment (start 133.448 98.2) (end 133.096 98.552) (width 0.254) (layer F.Cu) (net 4))
   (segment (start 133.448 92.101) (end 135.737 92.101) (width 0.254) (layer F.Cu) (net 4))
@@
   (segment (start 113.03 98.044) (end 113.03 98.044) (width 0.25) (layer B.Cu) (net 4))
   (segment (start 108.37 77.23) (end 110.91 77.23) (width 0.25) (layer F.Cu) (net 4))
+  (segment (start 118.11 98.401) (end 118.11 97.79) (width 0.25) (layer F.Cu) (net 5) (status 400000))
+  (segment (start 114.808 95.504) (end 113.03 95.504) (width 0.25) (layer F.Cu) (net 5) (status 800000))
+  (segment (start 116.078 96.774) (end 114.808 95.504) (width 0.25) (layer F.Cu) (net 5))
+  (segment (start 117.094 96.774) (end 116.078 96.774) (width 0.25) (layer F.Cu) (net 5))
+  (segment (start 118.11 97.79) (end 117.094 96.774) (width 0.25) (layer F.Cu) (net 5))
   (segment (start 144.78 102.846) (end 144.78 104.902) (width 0.254) (layer F.Cu) (net 5))
   (via (at 144.78 104.902) (size 0.6) (drill 0.4) (layers F.Cu B.Cu) (net 5))
@@
   (segment (start 132.334 96.012) (end 131.826 96.52) (width 0.254) (layer F.Cu) (net 5))
   (via (at 131.826 96.52) (size 0.6) (drill 0.4) (layers F.Cu B.Cu) (net 5))
+  (segment (start 121.539 98.401) (end 119.888 98.401) (width 0.254) (layer F.Cu) (net 5))
+  (segment (start 119.888 98.401) (end 118.11 98.401) (width 0.254) (layer F.Cu) (net 5))
   (segment (start 112.903 106.553) (end 112.903 106.68) (width 0.25) (layer F.Cu) (net 6))
   (segment (start 112.903 106.68) (end 111.379 108.204) (width 0.381) (layer F.Cu) (net 6))
@@
   (segment (start 154.686 91.948) (end 153.924 92.71) (width 0.254) (layer F.Cu) (net 24))
   (segment (start 153.924 92.71) (end 152.4 92.71) (width 0.254) (layer F.Cu) (net 24))
-  (segment (start 121.539 98.401) (end 118.11 98.401) (width 0.254) (layer F.Cu) (net 25))
-  (segment (start 149.86 95.25) (end 149.86 97.79) (width 0.254) (layer F.Cu) (net 26))
-  (segment (start 147.804 99.846) (end 144.78 99.846) (width 0.254) (layer F.Cu) (net 26))
-  (segment (start 149.86 97.79) (end 147.804 99.846) (width 0.254) (layer F.Cu) (net 26))
-  (segment (start 139.348 90.801) (end 141.601 90.801) (width 0.254) (layer F.Cu) (net 27))
-  (segment (start 143.51 92.71) (end 149.86 92.71) (width 0.254) (layer F.Cu) (net 27))
-  (segment (start 141.601 90.801) (end 143.51 92.71) (width 0.254) (layer F.Cu) (net 27))
-  (segment (start 139.348 90.801) (end 139.225 90.678) (width 0.254) (layer F.Cu) (net 27))
-  (segment (start 152.4 95.25) (end 152.4 97.79) (width 0.762) (layer F.Cu) (net 28))
+  (segment (start 149.86 95.25) (end 149.86 97.79) (width 0.254) (layer F.Cu) (net 25))
+  (segment (start 147.804 99.846) (end 144.78 99.846) (width 0.254) (layer F.Cu) (net 25))
+  (segment (start 149.86 97.79) (end 147.804 99.846) (width 0.254) (layer F.Cu) (net 25))
+  (segment (start 139.348 90.801) (end 141.601 90.801) (width 0.254) (layer F.Cu) (net 26))
+  (segment (start 143.51 92.71) (end 149.86 92.71) (width 0.254) (layer F.Cu) (net 26))
+  (segment (start 141.601 90.801) (end 143.51 92.71) (width 0.254) (layer F.Cu) (net 26))
+  (segment (start 139.348 90.801) (end 139.225 90.678) (width 0.254) (layer F.Cu) (net 26))
+  (segment (start 152.4 95.25) (end 152.4 97.79) (width 0.762) (layer F.Cu) (net 27))
   (zone (net 4) (net_name +5V) (layer F.Cu) (hatch edge 0.508)
     (connect_pads (clearance 0.508))
