File: Electrical/Circuit Boards/Raspberry Pi HATs/ADC HAT/HAT.kicad_pcb (KiCad board)
At the start: 2 copper layers, 65 x 56 mm, 31 parts, among them J1 CONN_01X02, J10 CONN_01X03, J11 CONN_01X03, J12 CONN_01X03, J13 CONN_01X03, J14 CONN_01X03, J15 CONN_01X03, J16 CONN_01X03, J17 CONN_01X03, J18 CONN_01X03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

Commit message: Add I2C test point labels
Other:
- board text added: "SCL"
- board text added: "SDA"
Changed lines of the file:
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@@
     (area 90.114287 72.333 185.100001 136.350001)
     (thickness 1.6)
-    (drawings 61)
+    (drawings 63)
     (tracks 224)
     (zones 0)
@@
     (descr "Through hole straight pin header, 1x02, 2.54mm pitch, single row")
     (tags "Through hole pin header THT 1x02 2.54mm single row")
-    (fp_text reference J1 (at 0 -2.33 90) (layer F.SilkS)
+    (fp_text reference J1 (at 0 -2.33 90) (layer F.SilkS) hide
       (effects (font (size 1 1) (thickness 0.15)))
     )
@@
     )
   )
+  (gr_text SCL (at 117.348 84.074) (layer F.SilkS)
+    (effects (font (size 1.5 1.5) (thickness 0.3)))
+  )
+  (gr_text SDA (at 106.68 84.074) (layer F.SilkS)
+    (effects (font (size 1.5 1.5) (thickness 0.3)))
+  )
   (gr_text "Only attach when\nVREF is grounded" (at 152.4 109.728 270) (layer F.SilkS)
